File: power.kicad_sch (KiCad schematic)
At the start: 6 parts

Commit message: Various updates
Parts:
- removed D4: PWR_LED, symbol Device:LED
- removed H1, H2, H3, H4: MhPad, symbol MyLib:MhPad
- removed R4: 500, symbol MyLib:R
