File: STM32H7-pill-hw.kicad_sch (KiCad schematic)
At the start: 0 parts

Commit message: Various updates
Other:
- removed sheet IO pins
- removed sheet User IOs
Changed lines of the file:
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@@
 	(paper "A4")
 	(sheet
-		(at 50.8 25.4)
-		(size 25.4 38.1)
+		(at 28.575 126.365)
+		(size 34.925 38.735)
 		(fields_autoplaced yes)
 		(stroke
@@
 		)
 		(property "Sheetname" "Power"
-			(at 50.8 24.6884 0)
+			(at 28.575 125.6534 0)
 			(effects
 				(font
@@
 		)
 		(property "Sheetfile" "power.kicad_sch"
-			(at 50.8 64.0846 0)
+			(at 28.575 165.6846 0)
 			(effects
 				(font
@@
 		)
 		(instances
-			(project "STM32h5-pill-hw"
+			(project "STM32H7-pill-hw"
 				(path "/32a39ea4-b179-4c09-9721-817d0177aae9"
 					(page "3")
@@
 	)
 	(sheet
-		(at 50.8 127)
-		(size 25.4 38.1)
-		(fields_autoplaced yes)
-		(stroke
-			(width 0.1524)
-			(type solid)
-		)
-		(fill
-			(color 0 0 0 0.0000)
-		)
-		(property "Sheetname" "User IOs"
-			(at 50.8 126.2884 0)
-			(effects
-				(font
-					(size 1.27 1.27)
-				)
-				(justify left bottom)
-			)
-		)
-		(property "Sheetfile" "untitled.kicad_sch"
-			(at 50.8 165.6846 0)
-			(effects
-				(font
-					(size 1.27 1.27)
-				)
-				(justify left top)
-			)
-		)
-		(instances
-			(project "STM32h5-pill-hw"
-				(path "/32a39ea4-b179-4c09-9721-817d0177aae9"
-					(page "6")
-				)
-			)
-		)
-	)
-	(sheet
-		(at 203.2 101.6)
-		(size 25.4 50.8)
+		(at 192.405 98.425)
+		(size 43.18 63.5)
 		(fields_autoplaced yes)
 		(stroke
@@
 		)
 		(property "Sheetname" "Sensors"
-			(at 203.2 100.8884 0)
+			(at 192.405 97.7134 0)
 			(effects
 				(font
@@
 		)
 		(property "Sheetfile" "sensors.kicad_sch"
-			(at 203.2 152.9846 0)
+			(at 192.405 162.5096 0)
 			(effects
 				(font
@@
 		)
 		(instances
-			(project "STM32h5-pill-hw"
+			(project "STM32H7-pill-hw"
 				(path "/32a39ea4-b179-4c09-9721-817d0177aae9"
 					(page "5")
@@
 	)
 	(sheet
-		(at 203.2 38.1)
-		(size 25.4 50.8)
+		(at 28.575 24.765)
+		(size 34.925 95.25)
 		(fields_autoplaced yes)
 		(stroke
@@
 		)
 		(property "Sheetname" "Interfaces"
-			(at 203.2 37.3884 0)
+			(at 28.575 24.0534 0)
 			(effects
 				(font
@@
 		)
 		(property "Sheetfile" "interfaces.kicad_sch"
-			(at 203.2 89.4846 0)
+			(at 28.575 120.5996 0)
 			(effects
 				(font
@@
 		)
 		(instances
-			(project "STM32h5-pill-hw"
+			(project "STM32H7-pill-hw"
 				(path "/32a39ea4-b179-4c09-9721-817d0177aae9"
 					(page "7")
@@
 	)
 	(sheet
-		(at 50.8 76.2)
-		(size 25.4 38.1)
-		(fields_autoplaced yes)
-		(stroke
-			(width 0.1524)
-			(type solid)
-		)
-		(fill
-			(color 0 0 0 0.0000)
-		)
-		(property "Sheetname" "IO pins"
-			(at 50.8 75.4884 0)
-			(effects
-				(font
-					(size 1.27 1.27)
-				)
-				(justify left bottom)
-			)
-		)
-		(property "Sheetfile" "IO_pins.kicad_sch"
-			(at 50.8 114.8846 0)
-			(effects
-				(font
-					(size 1.27 1.27)
-				)
-				(justify left top)
-			)
-		)
-		(instances
-			(project "STM32h5-pill-hw"
-				(path "/32a39ea4-b179-4c09-9721-817d0177aae9"
-					(page "4")
-				)
-			)
-		)
-	)
-	(sheet
-		(at 114.3 25.4)
-		(size 50.8 139.7)
+		(at 88.9 24.765)
+		(size 50.8 140.335)
 		(fields_autoplaced yes)
 		(stroke
@@
 		)
 		(property "Sheetname" "MCU"
-			(at 114.3 24.6884 0)
+			(at 88.9 24.0534 0)
 			(effects
 				(font
@@
 		)
 		(property "Sheetfile" "MCU.kicad_sch"
-			(at 114.3 165.6846 0)
+			(at 88.9 165.6846 0)
 			(effects
 				(font
@@
 		)
 		(instances
-			(project "STM32h5-pill-hw"
+			(project "STM32H7-pill-hw"
 				(path "/32a39ea4-b179-4c09-9721-817d0177aae9"
 					(page "2")

Commit message: Updates
Other:
- sheet Interfaces ports: added USBD+, USBD-; removed none
Changed lines of the file:
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@@
+			)
+		)
+		(pin "USBD-" output
+			(at 63.5 71.12 0)
+			(effects
+				(font
+					(size 1.27 1.27)
+				)
+				(justify right)
+			)
+		)
+		(pin "USBD+" output
+			(at 63.5 68.58 0)
+			(effects
+				(font
+					(size 1.27 1.27)
+				)
+				(justify right)
 			)
 		)
