File: interfaces.kicad_sch (KiCad schematic)
At the start: 3 parts, among them J1 USB_C_Connector_16P, J2 Conn_02x03_Top_Bottom, U3 USBLC6-2P6

Commit message: Various updates
Parts:
- removed J1: USB_C_Connector_16P, symbol MyLib:USB_C_Connector_16P
- removed J2: Conn_02x03_Top_Bottom, symbol Connector_Generic:Conn_02x03_Top_Bottom
- removed U3: USBLC6-2P6, Package_TO_SOT_SMD:SOT-666, symbol MyLib:USBLC6-2P6
- added J1: USB_C_Connector_16P, symbol AetherLib:USB_C_Connector_16P
- added J2: SD_CARD, symbol Connector:Micro_SD_Card
- added J3: Conn_ST_STDC14, symbol Connector:Conn_ST_STDC14
- added R15, R16: 5.1k, symbol AetherLib:R
- added R17, R18: 22, symbol AetherLib:R
- added U3: USBLC6-2P6, Package_TO_SOT_SMD:SOT-666, symbol Power_Protection:USBLC6-2P6
Connections:
- net SWCLK: now also J3.6 (JCLK/SWCLK)
- net SWDIO: now also J3.4 (JTMS/SWDIO)
- new net: J1.B5 (CC2), R15.1
- new net: J1.A5 (CC1), R16.1
- new net: R18.1, U3.4 (I/O2)
- new net: R17.1, U3.6 (I/O1)
- new net 3V3: J2.4 (VDD), J3.3 (VCC)
- new net 5Vbus: J1.A4 (VBUS), J1.A9 (VBUS), J1.B4 (VBUS), J1.B9 (VBUS), U3.5 (VBUS)
- new net GND: J1.A1 (GND), J1.A12 (GND), J1.B1 (GND), J1.B12 (GND), J1.S1 (SHIELD), J2.6 (VSS), J3.11 (GNDDetect), J3.5 (GND), J3.7 (GND), R15.2, R16.2, U3.2 (GND)
- new net NRST: J3.12 (~{RST})
- new net RAW_USBD+: J1.A6 (D+), J1.B6 (D+), U3.3 (I/O2)
- new net RAW_USBD-: J1.A7 (D-), J1.B7 (D-), U3.1 (I/O1)
- new net SD_CLK: J2.5 (CLK)
- new net SD_CMD: J2.3 (CMD)
- new net SD_D0: J2.7 (DAT0)
- new net SD_D1: J2.8 (DAT1)
- new net SD_D2: J2.1 (DAT2)
- new net SD_D3: J2.2 (DAT3/CD)
- new net SWO: J3.8 (JTDO/SWO)
- new net USBD+: R18.2
- new net USBD-: R17.2
- new net VCP_UART_RX: J3.13 (VCP_RX)
- new net VCP_UART_TX: J3.14 (VCP_TX)
- no-connect marks 0 -> 2

Commit message: Updates
Parts:
- removed J2: SD_CARD, symbol Connector:Micro_SD_Card
- added J4: Micro_SD_Card_Det1, symbol Connector:Micro_SD_Card_Det1
Connections:
- net GND: now also J4.10 (SHIELD), J4.6 (VSS)
- net SD_CLK: now also J4.5 (CLK)
- net SD_CMD: now also J4.3 (CMD)
- net SD_D0: now also J4.7 (DAT0)
- net SD_D1: now also J4.8 (DAT1)
- net SD_D2: now also J4.1 (DAT2)
- net SD_D3: now also J4.2 (DAT3/CD)
- new net SD_DTCT: J4.9 (DET)
